File: hardware/ACDC_TUNS700F.kicad_pcb (KiCad board)
At the start: 2 copper layers, 217 x 67.5 mm, 14 parts, among them U1 TUNS700F28

Commit message: reference schematic complete
Parts:
- added C20: 680nF, Capacitor_THT:C_Rect_L18.0mm_W8.0mm_P15.00mm_FKS3_FKP3, B.Cu at (175.5, 33.0)
- added C21: 2x680nF, Capacitor_THT:C_Rect_L18.0mm_W8.0mm_P15.00mm_FKS3_FKP3, B.Cu at (175.5, 23.4)
- added C30: 680nF, Capacitor_THT:C_Rect_L18.0mm_W8.0mm_P15.00mm_FKS3_FKP3, B.Cu at (211.5, 23.9)
- added C31: 2x680nF, Capacitor_THT:C_Rect_L18.0mm_W8.0mm_P15.00mm_FKS3_FKP3, B.Cu at (211.5, 33.5)
- added C40: 10uF, Capacitor_SMD:C_1206_3216Metric_Pad1.33x1.80mm_HandSolder, F.Cu at (232.0, 40.9)
- added Cbc1: 2x390uF, Capacitor_THT:CP_Radial_D30.0mm_P10.00mm_SnapIn, B.Cu at (398.5, 39.5)
- added Cbc2: 2x390uF, Capacitor_THT:CP_Radial_D30.0mm_P10.00mm_SnapIn, B.Cu at (398.5, 71.0)
- added Co1: 1mF, Capacitor_THT:CP_Radial_D16.0mm_P7.50mm, F.Cu at (234.5, 30.4)
- added GD1: GDT_2Pin, ACDC_TUNS700F:GDT_2093-300-SM-RPLF, B.Cu at (205.5, 88.0)
- added R1: 68k, Resistor_SMD:R_1206_3216Metric_Pad1.30x1.75mm_HandSolder, F.Cu at (123.5, 45.5)
- added R2: 68k, Resistor_SMD:R_1206_3216Metric_Pad1.30x1.75mm_HandSolder, F.Cu at (123.5, 50.5)
- added R3: 68k, Resistor_SMD:R_1206_3216Metric_Pad1.30x1.75mm_HandSolder, F.Cu at (123.5, 55.5)
- added R4: 68k, Resistor_SMD:R_1206_3216Metric_Pad1.30x1.75mm_HandSolder, F.Cu at (126.0, 45.5)
- added R5: 68k, Resistor_SMD:R_1206_3216Metric_Pad1.30x1.75mm_HandSolder, F.Cu at (126.0, 50.5)
- added R6: 68k, Resistor_SMD:R_1206_3216Metric_Pad1.30x1.75mm_HandSolder, F.Cu at (126.0, 55.5)
- added SK11: 620V, ACDC_TUNS700F:RV_Disc_D15,5mm_W7,1mm_P7,5mm, B.Cu at (169.0, 65.5)
- added SK21: 620V, ACDC_TUNS700F:RV_Disc_D15,5mm_W7,1mm_P7,5mm, B.Cu at (224.0, 88.0)
- added SK22: 620V, ACDC_TUNS700F:RV_Disc_D15,5mm_W7,1mm_P7,5mm, B.Cu at (232.5, 88.0)
- moved CY1 261.2 mm to (348.5, 90.0), turned to 180 degrees
- moved L2 173.8 mm to (229.0, 65.5)
- moved CY2 153.2 mm to (212.5, 48.0), turned to 90 degrees
- moved CY3 146.1 mm to (212.5, 83.0), turned to -90 degrees
- moved CX1 143.2 mm to (179.5, 65.5)
- moved CX2 141.6 mm to (212.5, 65.5)
- moved C11 140.0 mm to (249.0, 65.5)
- moved U1 137.6 mm to (319.0, 56.5)
- moved L1 111.1 mm to (196.0, 65.5)
- moved F1 84.7 mm to (187.5, 85.5)
- renumbered C1 to C11, CY3 to CY2, CY2 to CY3, L11 to L1, L12 to L2
Connections:
- net Net-(U1--BC) renamed -BC
- C11 pad 1: Net-(U1-AC1) -> AC1
- C11 pad 2: Net-(U1-AC2) -> AC2
- CX1 pad 1: unconnected-(CX1-Pad1) -> Net-(CX1-Pad1)
- CX2 pad 1: unconnected-(CX2-Pad1) -> Net-(CX2-Pad1)
- CY2 pad 1: unconnected-(CY3-Pad1) -> Net-(CX2-Pad2)
- CY2 pad 2: unconnected-(CY3-Pad2) -> FG
- CY3 pad 1: unconnected-(CY2-Pad1) -> Net-(CX2-Pad1)
- CY3 pad 2: unconnected-(CY2-Pad2) -> FG
- F1 pad 1: unconnected-(F1-Pad1) -> Net-(J1-Pin_1)
- F1 pad 2: unconnected-(F1-Pad2) -> Net-(CX1-Pad1)
- L1 pad 1: unconnected-(L11-Pad1) -> Net-(CX1-Pad1)
- L1 pad 2: unconnected-(L11-Pad2) -> Net-(J2-Pin_1)
- L1 pad 3: unconnected-(L11-Pad3) -> Net-(CX2-Pad2)
- L1 pad 4: unconnected-(L11-Pad4) -> Net-(CX2-Pad1)
- L2 pad 1: unconnected-(L12-Pad1) -> Net-(CX2-Pad1)
- L2 pad 2: unconnected-(L12-Pad2) -> Net-(CX2-Pad2)
- L2 pad 3: unconnected-(L12-Pad3) -> AC2
- L2 pad 4: unconnected-(L12-Pad4) -> AC1
- U1 pad 1: Net-(U1-AC1) -> AC1
- U1 pad 2: Net-(U1-AC2) -> AC2
- U1 pad 3: unconnected-(U1-R-Pad3) -> R
- U1 pad 4: unconnected-(U1-+BC-Pad4) -> +BC
- U1 pad 6: unconnected-(U1-+VOUT-Pad6) -> Net-(U1-+S)
- U1 pad 7: unconnected-(U1--VOUT-Pad7) -> Net-(U1--S)
- U1 pad 8: unconnected-(U1--S-Pad8) -> Net-(U1--S)
- U1 pad 9: unconnected-(U1-+S-Pad9) -> Net-(U1-+S)
Other:
- board outline removed

Commit message: board layout updates
Parts:
- added G***: LOGO, LOGO, F.Cu at (184.0, 81.5)
- added J1: Screw_Terminal_01x03, ACDC_TUNS700F:terminal_NC6-P108-03, F.Cu at (72.4, 76.2)
- added J2: +VO, TerminalBlock_Wuerth:Wuerth_REDCUBE-THR_WP-THRSH_74651194_THR, F.Cu at (254.5, 101.0)
- added J3: -VO, TerminalBlock_Wuerth:Wuerth_REDCUBE-THR_WP-THRSH_74651194_THR, F.Cu at (254.5, 66.5)
- added J4: Conn_01x04_Pin, Connector_PinHeader_2.54mm:PinHeader_1x04_P2.54mm_Vertical, F.Cu at (257.5, 125.0)
- added TFR1: 10R 139°C, ACDC_TUNS700F:TFR_DFP10112, F.Cu at (132.7, 120.0)
- C11, C20, C21, C30, C31, CX1, CX2, CY2, CY3, Cbc1, Cbc2, F1, GD1, L1, L2, SK11, SK21, SK22: moved to F.Cu
- C40, R1, R2, R3, R4, R5, R6, U1: moved to B.Cu
- moved Cbc2 231.7 mm to (172.7, 123.0), turned to -90 degrees
- moved H2 198.6 mm to (258.5, 139.0)
- moved Cbc1 184.7 mm to (233.7, 123.0), turned to -90 degrees
- moved H4 166.3 mm to (258.5, 54.0)
- moved CY2 155.5 mm to (82.0, 132.5), turned to 0 degrees
- moved CY1 147.2 mm to (209.5, 138.4)
- moved U1 134.6 mm to (186.6, 80.7)
- moved SK22 133.7 mm to (106.3, 132.1), turned to -90 degrees
- moved C11 132.2 mm to (116.8, 70.0), turned to -90 degrees
- moved L1 128.6 mm to (78.7, 118.1), turned to 180 degrees
- moved L2 121.3 mm to (111.8, 96.5), turned to 0 degrees
- moved H1 118.5 mm to (68.5, 139.0)
- moved SK21 118.2 mm to (114.3, 132.1)
- moved CX2 113.1 mm to (110.5, 114.3), turned to 0 degrees
- moved CY3 111.1 mm to (102.9, 65.0), turned to 180 degrees
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Connections:
- net Net-(U1-+S) renamed /+VO
- net Net-(U1--S) renamed /-VO
- U1 pad 10: unconnected-(U1-TRM-Pad10) -> Net-(J4-Pin_2)
- U1 pad 11: unconnected-(U1-IOG-Pad11) -> Net-(J4-Pin_1)
- U1 pad 12: unconnected-(U1-FG-Pad12) -> FG
Routing:
- net +BC: track 0.00 -> 162.7 mm
- net -BC: track 0.00 -> 146.3 mm
- net AC1: track 0.00 -> 111.9 mm
- net /-VO: track 0.00 -> 101.7 mm
- net AC2: track 0.00 -> 85.6 mm
- net Net-(CX2-Pad2): track 0.00 -> 78.0 mm
- net Net-(CX2-Pad1): track 0.00 -> 73.4 mm
- net Net-(J1-Pin_2): track 0.00 -> 65.3 mm
- net /+VO: track 0.00 -> 51.3 mm
- net Net-(CX1-Pad1): track 0.00 -> 47.4 mm
- net R: track 0.00 -> 37.8 mm
- net Net-(J4-Pin_2): track 0.00 -> 37.3 mm
- net Net-(J4-Pin_1): track 0.00 -> 35.8 mm
- net Net-(J1-Pin_1): track 0.00 -> 17.6 mm
- net Net-(GD1-Pad3): track 0.00 -> 15.1 mm
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- added copper zone on B.Cu, net /+VO
- added copper zone on F.Cu, net /+VO
- added copper zone on B.Cu, net /-VO
- added copper zone on F.Cu, net /-VO
- added copper zone on B.Cu, net FG
- added copper zone on F.Cu, net FG
Other:
- board outline added: 200 x 95 mm
- board text added: "+VO"
- board text added: "-VO"
- board text added: "28V 25A OUT"
- board text added: "700W AC/DC"
- board text added: "IOG"
- board text added: "January 2025"
- board text added: "Remi De Coster"
- board text added: "TRM"

Commit message: media uploads
Other:
- board text added: "+"
- board text added: "-"
Changed lines of the file:
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@@
 		(tags "C Disc series Radial pin pitch 10.00mm  diameter 9mm width 5.0mm Capacitor")
 		(property "Reference" "CY3"
-			(at 5 -3.75 360)
+			(at 5 -3.75 0)
 			(layer "F.SilkS")
 			(effects
@@
 		)
 		(property "Value" "2.2nF"
-			(at 5 3.75 360)
+			(at 5 3.75 0)
 			(layer "F.Fab")
 			(effects
@@
 		(tags "C Disc series Radial pin pitch 10.00mm  diameter 9mm width 5.0mm Capacitor")
 		(property "Reference" "CY2"
-			(at 5 -3.75 360)
+			(at 5 -3.75 0)
 			(layer "F.SilkS")
 			(effects
@@
 		)
 		(property "Value" "2.2nF"
-			(at 5 3.75 360)
+			(at 5 3.75 0)
 			(layer "F.Fab")
 			(effects
@@
 		)
 		(fp_text user "${REFERENCE}"
-			(at 5 0 360)
+			(at 5 0 0)
 			(layer "F.Fab")
 			(effects
@@
 		(tags "C Disc series Radial pin pitch 10.00mm  diameter 9mm width 5.0mm Capacitor")
 		(property "Reference" "CY1"
-			(at 5 -3.75 360)
+			(at 5 -3.75 0)
 			(layer "F.SilkS")
 			(effects
@@
 		)
 		(property "Value" "2.2nF"
-			(at 5 3.75 360)
+			(at 5 3.75 0)
 			(layer "B.Fab")
 			(effects
@@
 		)
 		(fp_text user "${REFERENCE}"
-			(at 5 0 360)
+			(at 5 0 0)
 			(layer "F.Fab")
 			(effects
@@
 		(tags "resistor handsolder")
 		(property "Reference" "R3"
-			(at 0 1.82 360)
+			(at 0 1.82 0)
 			(layer "B.SilkS")
 			(effects
@@
 		)
 		(property "Value" "68k"
-			(at 0 -1.82 360)
+			(at 0 -1.82 0)
 			(layer "B.Fab")
 			(effects
@@
 		)
 		(fp_text user "${REFERENCE}"
-			(at 0 0 360)
+			(at 0 0 0)
 			(layer "B.Fab")
 			(effects
@@
 		(tags "resistor handsolder")
 		(property "Reference" "R1"
-			(at 0 1.82 360)
+			(at 0 1.82 0)
 			(layer "B.SilkS")
 			(effects
@@
 		)
 		(property "Value" "68k"
-			(at 0 -1.82 360)
+			(at 0 -1.82 0)
 			(layer "B.Fab")
 			(effects
@@
 		)
 		(fp_text user "${REFERENCE}"
-			(at 0 0 360)
+			(at 0 0 0)
 			(layer "B.Fab")
 			(effects
@@
 		(tags "resistor handsolder")
 		(property "Reference" "R6"
-			(at 0 1.82 360)
+			(at 0 1.82 0)
 			(layer "B.SilkS")
 			(effects
@@
 		)
 		(property "Value" "68k"
-			(at 0 -1.82 360)
+			(at 0 -1.82 0)
 			(layer "B.Fab")
 			(effects
@@
 		)
 		(fp_text user "${REFERENCE}"
-			(at 0 0 360)
+			(at 0 0 0)
 			(layer "B.Fab")
 			(effects
@@
 		(tags "resistor handsolder")
 		(property "Reference" "R4"
-			(at 0 1.82 360)
+			(at 0 1.82 0)
 			(layer "B.SilkS")
 			(effects
@@
 		)
 		(property "Value" "68k"
-			(at 0 -1.82 360)
+			(at 0 -1.82 0)
 			(layer "B.Fab")
 			(effects
@@
 		)
 		(fp_text user "${REFERENCE}"
-			(at 0 0 360)
+			(at 0 0 0)
 			(layer "B.Fab")
 			(effects
@@
 		(tags "resistor handsolder")
 		(property "Reference" "R5"
-			(at 0 1.82 360)
+			(at 0 1.82 0)
 			(layer "B.SilkS")
 			(effects
@@
 		)
 		(property "Value" "68k"
-			(at 0 -1.82 360)
+			(at 0 -1.82 0)
 			(layer "B.Fab")
 			(effects
@@
 		)
 		(fp_text user "${REFERENCE}"
-			(at 0 0 360)
+			(at 0 0 0)
 			(layer "B.Fab")
 			(effects
@@
 		(tags "resistor handsolder")
 		(property "Reference" "R2"
-			(at 0 1.82 360)
+			(at 0 1.82 0)
 			(layer "B.SilkS")
 			(effects
@@
 		)
 		(property "Value" "68k"
-			(at 0 -1.82 360)
+			(at 0 -1.82 0)
 			(layer "B.Fab")
 			(effects
@@
 		)
 		(fp_text user "${REFERENCE}"
-			(at 0 0 360)
+			(at 0 0 0)
 			(layer "B.Fab")
 			(effects
@@
 		)
 	)
+	(gr_text "-"
+		(at 250 56 0)
+		(layer "F.SilkS")
+		(effects
+			(font
+				(size 4 4)
+				(thickness 0.8)
+				(bold yes)
+			)
+		)
+	)
 	(gr_text "-VO"
 		(at 255 120 0)
@@
 		)
 	)
+	(gr_text "+"
+		(at 250 112 0)
+		(layer "F.SilkS")
+		(effects
+			(font
+				(size 4 4)
+				(thickness 0.8)
+				(bold yes)
+			)
+		)
+	)
 	(gr_text " 700W AC/DC "
 		(at 80 56 0)
@@
 		(priority 3)
 		(connect_pads yes
-			(clearance 2)
+			(clearance 1.5)
 		)
 		(min_thickness 0.25)
@@
 		(polygon
 			(pts
-				(xy 126.5 111.5) (xy 246 111.5) (xy 246 48.5) (xy 126.5 48.5)
+				(xy 126.5 111.5) (xy 246 111.5) (xy 246 86) (xy 240.5 80) (xy 237 80) (xy 237 60) (xy 246 60) (xy 246 48.5)
+				(xy 126.5 48.5)
 			)
 		)
@@
 				(xy 131 77.5) (xy 131 108.5) (xy 156 108.5) (xy 160 104.5) (xy 167.5 104.5) (xy 167.5 107.5) (xy 161 107.5)
 				(xy 160 108.5) (xy 178.5 108.5) (xy 178.5 105.5) (xy 184.5 99.5) (xy 204 99.5) (xy 213.5 108.5)
-				(xy 242.5 108.5) (xy 242.5 102.5) (xy 236.5 98.5) (xy 236.5 82) (xy 234.5 79.5) (xy 234.5 61) (xy 242 61)
+				(xy 242.5 108.5) (xy 242.5 102.5) (xy 236.5 98.5) (xy 236.5 82) (xy 234.5 79.5) (xy 234.5 60) (xy 242 60)
 				(xy 242 53)
 			)
